File: hardware/feather-wing-pmod.kicad_pcb (KiCad board)
At the start: 2 copper layers, 50.8 x 22.9 mm, 12 parts, among them J2 Conn_Left, J3 Conn_Right

Commit message: v1.0: ready for mfg
Parts:
- added SW1: SW_SPST, tom-mechanical:SW_Push_1P1T_NO_CK_KMR2, F.Cu at (135.5, 83.2)
Connections:
- J2 pad 1: /~RST~ -> !RST
Routing:
- net !RST: track 0.00 -> 32.0 mm, vias 0 -> 1
- net GND: track 21.7 -> 25.8 mm, vias 2 -> 3
- net /A5: track 22.9 -> 24.9 mm
- net /RX: track 36.6 -> 35.5 mm
Other:
- board text added: "1-4:SPI 7-8:I2C"
- board text added: "10"
- board text added: "11"
- board text added: "12"
- board text added: "13"
- board text added: "3V3"
- board text added: "5"
- board text added: "6"
- board text added: "9"
- board text added: "A0"
- board text added: "A1"
- board text added: "A2"
- board text added: "A3"
- board text added: "A4"
- board text added: "A5"
- board text added: "GND"
- board text added: "MISC"
- board text added: "RX"
- board text added: "Reset"
- board text added: "TX"
