File: hardware/feather-wing-pmod.kicad_pcb (KiCad board)
At the start: 2 copper layers, 50.8 x 22.9 mm, 13 parts, among them J2 Conn_Left, J3 Conn_Right, SW1 SW_SPST

Commit message: #1 Upgrade for kicad v6 and add BOM
Other:
- net class Default removed
